Commit message: chore: re created xacro file

File: urdf/test_snippets.urdf (robot description, URDF)
Before this commit: robot Test_Robot, 7 links, 6 joints
Links:
- added link imu, mass 0.05; collision box size=0.05 0.05 0.05; visual box size=0.05 0.05 0.05
- link front_castor: mass 0.05 -> 0.1
- link left_wheel: mass 0.1 -> 0.5
- link right_wheel: mass 0.1 -> 0.5
Joints:
- removed joint joint_chassis_front_camera
- removed joint joint_chassis_velodyne_lidar
- added joint joint_chassis_imu: type fixed, parent chassis, child imu, origin xyz=0 0 0.05 rpy=0 0 0
- added joint joint_front_camera_velodyne_lidar: type fixed, parent front_camera, child velodyne_lidar, origin xyz=0 0 0.15 rpy=0 0 0
- added joint joint_imu_front_camera: type fixed, parent imu, child front_camera, origin xyz=0.15 0 0.15 rpy=0 0 0

Commit message: chore: recreate test urdf

File: urdf/test_snippets.urdf (robot description, URDF)
Before this commit: robot Test_Robot, 8 links, 7 joints
Links:
- link chassis: mass 1 -> 5
