Commit message: fix: Robot Drift Issue
The robot was drifting slowly during simulation. The drift is suppressed by adjusting inertias of the robot components.

File: urdf/snippets.urdf.xacro (robot description, xacro)
@@ -80,5 +80,5 @@
         </joint>
     </xacro:macro>
-    <xacro:macro name="sensor_rgb_camera" params=" name:=cam parent:=chassis width:=640 height:=480 fps:=10 visulize:=true near:=0.01 far:=300 hfov:=60 xyz:='0 0 0'">
+    <xacro:macro name="sensor_rgb_camera" params=" name:=cam parent:=chassis width:=640 height:=480 fps:=10 visulize:=true near:=0.01 far:=100 hfov:=60 xyz:='0 0 0'">
         <xacro:shape_link name="${name}" type="box" m="0.05" w="0.05" l="0.05" h="0.05" rgba="1 0 0 1" color="Red"/>
         <xacro:shape_joint type="fixed" parent="${parent}" child="${name}" xyz="${xyz}"/>
@@ -413,5 +413,5 @@
                 <!-- Plugin update rate in Hz -->
                 <!-- <updateRate>${update_rate}</updateRate> -->
-                <updateRate>40</updateRate>
+                <updateRate>20</updateRate>
                 <!-- Name of left joint, defaults to `left_joint` -->
                 <leftJoint>${left}</leftJoint>
@@ -423,5 +423,5 @@
                 <wheelDiameter>${d}</wheelDiameter>
                 <!-- Wheel acceleration, in rad/s^2, defaults to 0.0 rad/s^2 -->
-                <wheelAcceleration>1.0</wheelAcceleration>
+                <wheelAcceleration>0.0</wheelAcceleration>
                 <!-- Maximum torque which the wheels can produce, in Nm, defaults to 5 Nm -->
                 <wheelTorque>1</wheelTorque>
@@ -444,5 +444,5 @@
                 <!-- Set to true to swap right and left wheels, defaults to true -->
                 <legacyMode>true</legacyMode>
-                <rosDebugLevel>false</rosDebugLevel>
+                <rosDebugLevel>true</rosDebugLevel>
                 <publishOdomTF>true</publishOdomTF>
                 <publishTf>1</publishTf>

File: urdf/test_snippets.urdf.xacro (robot description, xacro)
@@ -12,7 +12,7 @@
     <link name="base_link"/>
     <xacro:shape_link name="chassis" type="box" m="1" w="0.4" l="0.2" h="0.05" rgba="0 0 1 ${alpha}" color="Blue"/>
-    <xacro:shape_link name="left_wheel" type="cylinder" m="0.1" r="0.1" h="0.05" rgba="0 1 0 1" color="Green"/>
-    <xacro:shape_link name="right_wheel" type="cylinder" m="0.1" r="0.1" h="0.05" rgba="0 1 0 1" color="Green"/>
-    <xacro:shape_link name="front_castor" type="sphere" m="0.05" r="0.05" rgba="1 0 0 1" color="Red"/>
+    <xacro:shape_link name="left_wheel" type="cylinder" m="0.5" r="0.1" h="0.05" rgba="0 1 0 1" color="Green"/>
+    <xacro:shape_link name="right_wheel" type="cylinder" m="0.5" r="0.1" h="0.05" rgba="0 1 0 1" color="Green"/>
+    <xacro:shape_link name="front_castor" type="sphere" m="0.1" r="0.05" rgba="1 0 0 1" color="Red"/>
     <!-- Create Joints: -->
     <xacro:shape_joint type="fixed" parent="base_link" child="chassis" xyz="0.1 0 0"/>
@@ -23,7 +23,7 @@
     <!-- Add Sensors -->
     <xacro:robot_drive_diff chassis="base_link" left="joint_chassis_left_wheel" right="joint_chassis_right_wheel" l="0.25" d="0.1" cmdtopic="cmd_vel" odomtopic="odom"/>
-    <xacro:sensor_rgb_camera name="front_camera" parent="chassis" width="640" height="480" fps="10" xyz="0.15 0 0.05"/>
-    <xacro:sensor_lidar_3d name="velodyne_lidar" parent="chassis" topic="/velodyne_points" rate="20" noise="0" minRange="0.1" maxRange="100" samples="360" xyz="0.15 0 0.15" visulize="false"/>
-    <xacro:sensor_imu_ros name="imu" parent="chassis" topic="/imu" rate="20" noise="0" xyz="0.15 0 0.10" visulize="false"/>
+    <xacro:sensor_imu_ros name="imu" parent="chassis" topic="/imu" rate="20" noise="0" xyz="0 0 0.05" visulize="false"/>
+    <xacro:sensor_rgb_camera name="front_camera" parent="imu" width="640" height="480" fps="10" xyz="0.15 0 0.15"/>
+    <xacro:sensor_lidar_3d name="velodyne_lidar" parent="front_camera" topic="/velodyne_points" rate="20" noise="0" minRange="0.1" maxRange="100" samples="360" xyz="0 0 0.15" visulize="false"/>
     <!-- <xacro:sensor_stereo_camera name="stereo_camera" parent="chassis" width="640" height="480" fps="10" xyz="0.15 0 0.05"/> -->
     <!-- <xacro:sensor_depth_camera name="kinect_camera" parent="chassis" width="640" height="480" fps="10" xyz="0.15 0 0.05"/> -->

Commit message: feat: Add baseline to the stereo and kinect camera

File: urdf/snippets.urdf.xacro (robot description, xacro)
@@ -124,5 +124,5 @@
         </gazebo>
     </xacro:macro>
-    <xacro:macro name="sensor_stereo_camera" params=" name:=stereo parent:=chassis width:=640 height:=480 fps:=10 visulize:=true near:=0.01 far:=300 hfov:=60 xyz:='0 0 0'">
+    <xacro:macro name="sensor_stereo_camera" params=" name:=stereo parent:=chassis width:=640 height:=480 fps:=10 visulize:=true near:=0.01 far:=300 hfov:=60 xyz:='0 0 0' baseline:=0.07">
         <xacro:shape_link name="${name}" type="box" m="0.05" w="0.05" l="0.05" h="0.05" rgba="1 0 0 1" color="Red"/>
         <xacro:shape_joint type="fixed" parent="${parent}" child="${name}" xyz="${xyz}"/>
@@ -173,5 +173,5 @@
                     <cameraInfoTopicName>camera_info</cameraInfoTopicName>
                     <frameName>left_camera_optical_frame</frameName>
-                    <hackBaseline>0.07</hackBaseline>
+                    <hackBaseline>${baseline}</hackBaseline>
                     <distortionK1>0.0</distortionK1>
                     <distortionK2>0.0</distortionK2>
@@ -183,5 +183,5 @@
         </gazebo>
     </xacro:macro>
-    <xacro:macro name="sensor_depth_camera" params=" name:=stereo parent:=chassis width:=640 height:=480 fps:=10 visulize:=true near:=0.01 far:=300 hfov:=60 xyz:='0 0 0'">
+    <xacro:macro name="sensor_depth_camera" params=" name:=stereo parent:=chassis width:=640 height:=480 fps:=10 visulize:=true near:=0.01 far:=300 hfov:=60 xyz:='0 0 0' baseline:=0.1">
         <xacro:shape_link name="${name}" type="box" m="0.05" w="0.05" l="0.05" h="0.05" rgba="1 0 0 1" color="Red"/>
         <xacro:shape_joint type="fixed" parent="${parent}" child="${name}" xyz="${xyz}"/>
@@ -208,5 +208,5 @@
                 </camera>
                 <camera name="right">
-                    <pose>0 -0.07 0 0 0 0</pose>
+                    <pose>0 -${baseline} 0 0 0 0</pose>
                     <horizontal_fov>${radians(hfov)}</horizontal_fov>
                     <image>
@@ -226,5 +226,5 @@
                 </camera>
                 <plugin name="depth_camera_controller" filename="libgazebo_ros_openni_kinect.so">
-                    <baseline>0.2</baseline>
+                    <baseline>${baseline}</baseline>
                     <alwaysOn>true</alwaysOn>
                     <updateRate>${fps}</updateRate>

Commit message: feat: Add mesh tag to the shape_link macro

File: urdf/snippets.urdf.xacro (robot description, xacro)
@@ -26,13 +26,18 @@
         <visual>
             <geometry>
-                <xacro:if value="${type == 'box'}">
-                    <box size="${w} ${l} ${h}"/>
+                <xacro:if value="${mesh == ''}">
+                    <xacro:if value="${type == 'box'}">
+                        <box size="${w} ${l} ${h}"/>
+                    </xacro:if>
+                    <xacro:if value="${type == 'cylinder'}">
+                        <cylinder radius="${r}" length="${h}"/>
+                    </xacro:if>
+                    <xacro:if value="${type == 'sphere'}">
+                        <sphere radius="${r}"/>
+                    </xacro:if>
                 </xacro:if>
-                <xacro:if value="${type == 'cylinder'}">
-                    <cylinder radius="${r}" length="${h}"/>
-                </xacro:if>
-                <xacro:if value="${type == 'sphere'}">
-                    <sphere radius="${r}"/>
-                </xacro:if>
+                <xacro:unless value="${mesh == ''}">
+                    <mesh filename="${mesh}"/>
+                </xacro:unless>
             </geometry>
             <material name="${rgba}">
@@ -58,5 +63,5 @@
     </xacro:property>
     <!-- Shape Macro Link :w:x-axis, l:y-axis, h:z-axis, r:x-y plane -->
-    <xacro:macro name="shape_link" params="name:=MyRobot type:=box m:=1 w:=1 l:=1 h:=1 r:=1 rgba:='0 0 0 1' xyz='0 0 0' rpy='0 0 0' color:=Red">
+    <xacro:macro name="shape_link" params="name:=MyRobot type:=box m:=1 w:=1 l:=1 h:=1 r:=1 rgba:='0 0 0 1' xyz='0 0 0' rpy='0 0 0' color:=Red mesh:=''">
         <link name="${name}">
             <!-- <origin xyz="${xyz}" rpy="${rpy}"/> -->
@@ -65,7 +70,9 @@
             <xacro:insert_block name="shape_collision"/>
         </link>
-        <gazebo reference="${name}">
-            <material>Gazebo/${color}</material>
-        </gazebo>
+        <xacro:if value="${mesh == ''}">
+            <gazebo reference="${name}">
+                <material>Gazebo/${color}</material>
+            </gazebo>
+        </xacro:if>
     </xacro:macro>
     <!-- Create a joint: type=fixed|continuous|revolute|planner|floating -->

Commit message: fix: Update collision tag for mesh option

File: urdf/snippets.urdf.xacro (robot description, xacro)
@@ -50,13 +50,18 @@
         <collision>
             <geometry>
-                <xacro:if value="${type == 'box'}">
-                    <box size="${w} ${l} ${h}"/>
+                <xacro:if value="${mesh == ''}">
+                    <xacro:if value="${type == 'box'}">
+                        <box size="${w} ${l} ${h}"/>
+                    </xacro:if>
+                    <xacro:if value="${type == 'cylinder'}">
+                        <cylinder radius="${r}" length="${h}"/>
+                    </xacro:if>
+                    <xacro:if value="${type == 'sphere'}">
+                        <sphere radius="${r}"/>
+                    </xacro:if>
                 </xacro:if>
-                <xacro:if value="${type == 'cylinder'}">
-                    <cylinder radius="${r}" length="${h}"/>
-                </xacro:if>
-                <xacro:if value="${type == 'sphere'}">
-                    <sphere radius="${r}"/>
-                </xacro:if>
+                <xacro:unless value="${mesh == ''}">
+                    <mesh filename="${mesh}"/>
+                </xacro:unless>
             </geometry>
         </collision>

Commit message: docs: improve documentation of xacro files
undefined

File: urdf/snippets.urdf.xacro (robot description, xacro)
@@ -6,7 +6,8 @@
         Desciption: Xacro snippits for various URDF tags.
     -->
+    <!-- Common properties -->
     <xacro:property name="alpha" value="0.5"/>
     <!-- Property Block: Shape Inertia, w:x-axis, l:y-axis, h:z-axis, r:x-y plane -->
-    <xacro:property name="shape_inertial">
+     <xacro:property name="shape_inertial">
         <inertial>
             <mass value="${m}"/>
@@ -92,4 +93,6 @@
         </joint>
     </xacro:macro>
+    <!-- Sensor Macros -->
+    <!-- RGB Camera Sensor -->
     <xacro:macro name="sensor_rgb_camera" params=" name:=cam parent:=chassis width:=640 height:=480 fps:=10 visulize:=true near:=0.01 far:=100 hfov:=60 xyz:='0 0 0'">
         <xacro:shape_link name="${name}" type="box" m="0.05" w="0.05" l="0.05" h="0.05" rgba="1 0 0 1" color="Red"/>
@@ -136,4 +139,5 @@
         </gazebo>
     </xacro:macro>
+    <!-- Stereo Camera Sensor -->
     <xacro:macro name="sensor_stereo_camera" params=" name:=stereo parent:=chassis width:=640 height:=480 fps:=10 visulize:=true near:=0.01 far:=300 hfov:=60 xyz:='0 0 0' baseline:=0.07">
         <xacro:shape_link name="${name}" type="box" m="0.05" w="0.05" l="0.05" h="0.05" rgba="1 0 0 1" color="Red"/>
@@ -195,4 +199,5 @@
         </gazebo>
     </xacro:macro>
+    <!-- Depth Camera Sensor -->
     <xacro:macro name="sensor_depth_camera" params=" name:=stereo parent:=chassis width:=640 height:=480 fps:=10 visulize:=true near:=0.01 far:=300 hfov:=60 xyz:='0 0 0' baseline:=0.1">
         <xacro:shape_link name="${name}" type="box" m="0.05" w="0.05" l="0.05" h="0.05" rgba="1 0 0 1" color="Red"/>
@@ -264,4 +269,5 @@
         </gazebo>
     </xacro:macro>
+    <!-- Video Sensor -->
     <xacro:macro name="sensor_video" params="link:=chassis width:=160 height:=120 topic:=image">
         <gazebo reference="${link}">
@@ -275,4 +281,5 @@
         </gazebo>
     </xacro:macro>
+    <!-- Bumper Sensor -->
     <xacro:macro name="sensor_bumper" params="name:=bumper rate:=20 frame:=world">
         <gazebo>
@@ -285,4 +292,5 @@
         </gazebo>
     </xacro:macro>
+    <!-- IMU Sensor (Gazebo) -->
     <xacro:macro name="sensor_imu_gazebo" params="parent:=chassis name:=base_link topic:=imu rate:=20 noise:=0">
         <!-- IMU plugin, without gravity -->
@@ -302,4 +310,5 @@
         </gazebo>
     </xacro:macro>
+    <!-- IMU Sensor (ROS) -->
     <xacro:macro name="sensor_imu_ros" params="parent:=chassis name:=base_link topic:=imu rate:=20 noise:=0 xyz:='0 0 0' visulize:=true">
         <!-- IMU plugin, with gravity -->
@@ -326,4 +335,5 @@
         </gazebo>
     </xacro:macro>
+    <!-- 2D Laser Sensor -->
     <xacro:macro name="sensor_laser_2d" params="parent:=chassis name:=laser topic:=/scan rate:=20 noise:=0 minRange:=0.1 maxRange:=100 samples:=360 xyz:='0 0 0' visulize:=true">
         <xacro:shape_link name="${name}" type="box" m="0.05" w="0.05" l="0.05" h="0.05" rgba="1 0 0 1" color="Red"/>
@@ -366,4 +376,5 @@
         </gazebo>
     </xacro:macro>
+    <!-- 3D Lidar Sensor -->
     <xacro:macro name="sensor_lidar_3d" params="parent:=chassis name:=base_link topic:=/velodyne_points rate:=20 noise:=0 minRange:=0.1 maxRange:=100 samples:=360 xyz:='0 0 0' visulize:=true">
         <xacro:shape_link name="${name}" type="box" m="0.05" w="0.05" l="0.05" h="0.05" rgba="1 0 0 1" color="Red"/>
@@ -409,4 +420,6 @@
         </gazebo>
     </xacro:macro>
+    <!-- Actuator Macros -->
+    <!-- Castor Wheel Friction -->
     <xacro:macro name="castor_friction" params="name:=castor_wheel mu1:=0 mu2:=0 kp:=1e9 kd:=0 fdir:='0 0 0'">
         <gazebo reference="${name}">
@@ -419,4 +432,5 @@
         </gazebo>
     </xacro:macro>
+    <!-- Robot Drive Differential -->
     <xacro:macro name="robot_drive_diff" params="chassis:=base_link left:=joint_chassis_left_wheel right:=joint_chassis_right_wheel l:=0.25 d:=0.1 cmdtopic:=cmd_vel odomtopic:=odom">
         <gazebo>
@@ -462,4 +476,5 @@
         </gazebo>
     </xacro:macro>
+    <!-- Robot Drive Skid Steer -->
     <xacro:macro name="robot_drive_skid_steer" params="chassis:=base_link front_left:=joint_chassis_front_left_wheel front_right:=joint_chassis_front_right_wheel rear_left:=joint_chassis_rear_left_wheel rear_right:=joint_chassis_rear_right_wheel l:=0.25 d:=0.1 cmdtopic:=cmd_vel odomtopic:=odom">
         <gazebo>

File: urdf/test_snippets.urdf.xacro (robot description, xacro)
@@ -1,13 +1,14 @@
 <?xml version="1.0"?>
 <!--
-        Author: Dr. -Ing. Ahmad Kamal Nasir
-        Email: dringakn@gmail.com
-        Description: To Generate the URDF file, use the following command
-                     xacro test_snippets.urdf.xacro -o test_snippets.urdf
+    Author: Dr. -Ing. Ahmad Kamal Nasir
+    Email: dringakn@gmail.com
+    Description: This URDF file defines the robot model for a simulated robot named "Test_Robot."
+                 To generate the URDF file, use the following command:
+                 xacro test_snippets.urdf.xacro -o test_snippets.urdf
 -->
 <robot xmlns:xacro="http://www.ros.org/wiki/xacro" name="Test_Robot">
-    <!-- Include my custom URDF snippets for visual/inertia/links/joints tags -->
+    <!-- Include custom URDF snippets for visual, inertia, links, and joints tags -->
     <xacro:include filename="./snippets.urdf.xacro"/>
-    <!-- Create links: w:x-axis, l:y-axis, h:z-axis -->
+    <!-- Create robot links along the x, y, and z axes -->
     <link name="base_link"/>
     <xacro:shape_link name="chassis" type="box" m="1" w="0.4" l="0.2" h="0.05" rgba="0 0 1 ${alpha}" color="Blue"/>

Commit message: chore: change odmometery sensor update rate

File: urdf/snippets.urdf.xacro (robot description, xacro)
@@ -9,5 +9,5 @@
     <xacro:property name="alpha" value="0.5"/>
     <!-- Property Block: Shape Inertia, w:x-axis, l:y-axis, h:z-axis, r:x-y plane -->
-     <xacro:property name="shape_inertial">
+    <xacro:property name="shape_inertial">
         <inertial>
             <mass value="${m}"/>
@@ -439,5 +439,5 @@
                 <!-- Plugin update rate in Hz -->
                 <!-- <updateRate>${update_rate}</updateRate> -->
-                <updateRate>20</updateRate>
+                <updateRate>50</updateRate>
                 <!-- Name of left joint, defaults to `left_joint` -->
                 <leftJoint>${left}</leftJoint>
