Commit message: chore: correct typo (xacro variable: visualize)

File: urdf/snippets.urdf.xacro (robot description, xacro)
@@ -95,10 +95,10 @@
     <!-- Sensor Macros -->
     <!-- RGB Camera Sensor -->
-    <xacro:macro name="sensor_rgb_camera" params=" name:=cam parent:=chassis width:=640 height:=480 fps:=10 visulize:=true near:=0.01 far:=100 hfov:=60 xyz:='0 0 0'">
+    <xacro:macro name="sensor_rgb_camera" params=" name:=cam parent:=chassis width:=640 height:=480 fps:=10 visualize:=true near:=0.01 far:=100 hfov:=60 xyz:='0 0 0'">
         <xacro:shape_link name="${name}" type="box" m="0.05" w="0.05" l="0.05" h="0.05" rgba="1 0 0 1" color="Red"/>
         <xacro:shape_joint type="fixed" parent="${parent}" child="${name}" xyz="${xyz}"/>
         <gazebo reference="${name}">
             <sensor type="camera" name="camera_sensor">
-                <visualize>${visulize}</visualize>
+                <visualize>${visualize}</visualize>
                 <update_rate>${fps}</update_rate>
                 <camera name="head">
@@ -140,10 +140,10 @@
     </xacro:macro>
     <!-- Stereo Camera Sensor -->
-    <xacro:macro name="sensor_stereo_camera" params=" name:=stereo parent:=chassis width:=640 height:=480 fps:=10 visulize:=true near:=0.01 far:=300 hfov:=60 xyz:='0 0 0' baseline:=0.07">
+    <xacro:macro name="sensor_stereo_camera" params=" name:=stereo parent:=chassis width:=640 height:=480 fps:=10 visualize:=true near:=0.01 far:=300 hfov:=60 xyz:='0 0 0' baseline:=0.07">
         <xacro:shape_link name="${name}" type="box" m="0.05" w="0.05" l="0.05" h="0.05" rgba="1 0 0 1" color="Red"/>
         <xacro:shape_joint type="fixed" parent="${parent}" child="${name}" xyz="${xyz}"/>
         <gazebo reference="${name}">
             <sensor type="multicamera" name="stereo_camera">
-                <visualize>${visulize}</visualize>
+                <visualize>${visualize}</visualize>
                 <update_rate>${fps}</update_rate>
                 <camera name="left">
@@ -200,10 +200,10 @@
     </xacro:macro>
     <!-- Depth Camera Sensor -->
-    <xacro:macro name="sensor_depth_camera" params=" name:=stereo parent:=chassis width:=640 height:=480 fps:=10 visulize:=true near:=0.01 far:=300 hfov:=60 xyz:='0 0 0' baseline:=0.1">
+    <xacro:macro name="sensor_depth_camera" params=" name:=stereo parent:=chassis width:=640 height:=480 fps:=10 visualize:=true near:=0.01 far:=300 hfov:=60 xyz:='0 0 0' baseline:=0.1">
         <xacro:shape_link name="${name}" type="box" m="0.05" w="0.05" l="0.05" h="0.05" rgba="1 0 0 1" color="Red"/>
         <xacro:shape_joint type="fixed" parent="${parent}" child="${name}" xyz="${xyz}"/>
         <gazebo reference="${name}">
             <sensor type="depth" name="depth_camera">
-                <visualize>${visulize}</visualize>
+                <visualize>${visualize}</visualize>
                 <update_rate>${fps}</update_rate>
                 <camera name="kinect">
@@ -311,5 +311,5 @@
     </xacro:macro>
     <!-- IMU Sensor (ROS) -->
-    <xacro:macro name="sensor_imu_ros" params="parent:=chassis name:=base_link topic:=imu rate:=20 noise:=0 xyz:='0 0 0' visulize:=true">
+    <xacro:macro name="sensor_imu_ros" params="parent:=chassis name:=base_link topic:=imu rate:=20 noise:=0 xyz:='0 0 0' visualize:=true">
         <!-- IMU plugin, with gravity -->
         <xacro:shape_link name="${name}" type="box" m="0.05" w="0.05" l="0.05" h="0.05" rgba="1 0 0 1" color="Red"/>
@@ -318,5 +318,5 @@
             <gravity>true</gravity>
             <sensor name="imu_sensor" type="imu">
-                <visualize>${visulize}</visualize>
+                <visualize>${visualize}</visualize>
                 <always_on>true</always_on>
                 <update_rate>${rate}</update_rate>
@@ -336,5 +336,5 @@
     </xacro:macro>
     <!-- 2D Laser Sensor -->
-    <xacro:macro name="sensor_laser_2d" params="parent:=chassis name:=laser topic:=/scan rate:=20 noise:=0 minRange:=0.1 maxRange:=100 samples:=360 xyz:='0 0 0' visulize:=true">
+    <xacro:macro name="sensor_laser_2d" params="parent:=chassis name:=laser topic:=/scan rate:=20 noise:=0 minRange:=0.1 maxRange:=100 samples:=360 xyz:='0 0 0' visualize:=true">
         <xacro:shape_link name="${name}" type="box" m="0.05" w="0.05" l="0.05" h="0.05" rgba="1 0 0 1" color="Red"/>
         <xacro:shape_joint type="fixed" parent="${parent}" child="${name}" xyz="${xyz}"/>
@@ -343,5 +343,5 @@
             <sensor type="gpu_ray" name="front_laser_sensor">
                 <pose>0 0 0 0 0 0</pose>
-                <visualize>${visulize}</visualize>
+                <visualize>${visualize}</visualize>
                 <update_rate>${rate}</update_rate>
                 <ray>
@@ -377,10 +377,10 @@
     </xacro:macro>
     <!-- 3D Lidar Sensor -->
-    <xacro:macro name="sensor_lidar_3d" params="parent:=chassis name:=base_link topic:=/velodyne_points rate:=20 noise:=0 minRange:=0.1 maxRange:=100 samples:=360 xyz:='0 0 0' visulize:=true">
+    <xacro:macro name="sensor_lidar_3d" params="parent:=chassis name:=base_link topic:=/velodyne_points rate:=20 noise:=0 minRange:=0.1 maxRange:=100 samples:=360 xyz:='0 0 0' visualize:=true">
         <xacro:shape_link name="${name}" type="box" m="0.05" w="0.05" l="0.05" h="0.05" rgba="1 0 0 1" color="Red"/>
         <xacro:shape_joint type="fixed" parent="${parent}" child="${name}" xyz="${xyz}"/>
         <gazebo reference="${name}">
             <sensor type="gpu_ray" name="front_lidar-VLP16">
-                <visualize>${visulize}</visualize>
+                <visualize>${visualize}</visualize>
                 <update_rate>${rate}</update_rate>
                 <ray>

File: urdf/test_snippets.urdf.xacro (robot description, xacro)
@@ -24,7 +24,7 @@
     <!-- Add Sensors -->
     <xacro:robot_drive_diff chassis="base_link" left="joint_chassis_left_wheel" right="joint_chassis_right_wheel" l="0.25" d="0.1" cmdtopic="cmd_vel" odomtopic="odom"/>
-    <xacro:sensor_imu_ros name="imu" parent="chassis" topic="/imu" rate="20" noise="0" xyz="0 0 0.05" visulize="false"/>
+    <xacro:sensor_imu_ros name="imu" parent="chassis" topic="/imu" rate="20" noise="0" xyz="0 0 0.05" visualize="false"/>
     <xacro:sensor_rgb_camera name="front_camera" parent="imu" width="640" height="480" fps="10" xyz="0.15 0 0.15"/>
-    <xacro:sensor_lidar_3d name="velodyne_lidar" parent="front_camera" topic="/velodyne_points" rate="20" noise="0" minRange="0.1" maxRange="100" samples="360" xyz="0 0 0.15" visulize="false"/>
+    <xacro:sensor_lidar_3d name="velodyne_lidar" parent="front_camera" topic="/velodyne_points" rate="20" noise="0" minRange="0.1" maxRange="100" samples="360" xyz="0 0 0.15" visualize="false"/>
     <!-- <xacro:sensor_stereo_camera name="stereo_camera" parent="chassis" width="640" height="480" fps="10" xyz="0.15 0 0.05"/> -->
     <!-- <xacro:sensor_depth_camera name="kinect_camera" parent="chassis" width="640" height="480" fps="10" xyz="0.15 0 0.05"/> -->

Commit message: feat: tricycle drive plugin xacro

File: urdf/snippets.urdf.xacro (robot description, xacro)
@@ -520,4 +520,52 @@
         </gazebo>
     </xacro:macro>
+    <!-- Tricycle Drive:
+    The tricycle drive is typically used for robots with
+    one front steering wheel and two rear driving wheels,
+    similar to how a tricycle or a front-steering robot works -->
+    <xacro:macro name="robot_drive_tricycle" params="
+        chassis:=base_link
+        steering_joint:=front_steering_joint
+        drive_joint_left:=joint_rear_left_wheel
+        drive_joint_right:=joint_rear_right_wheel
+        wheelbase:=0.8
+        wheel_radius:=0.15
+        steering_limit:=0.78539816339  # ~45 degrees in radians
+        cmdtopic:=/cmd_vel
+        odomtopic:=/odom
+        update_rate:=50">
+        <gazebo>
+            <!-- Tricycle Drive Plugin -->
+            <plugin name="tricycle_drive_controller" filename="libgazebo_ros_tricycle_drive.so">
+                <!-- Name of the front steering joint -->
+                <steeringJoint>${steering_joint}</steeringJoint>
+                <!-- Names of the rear left and right drive joints -->
+                <driveLeftJoint>${drive_joint_left}</driveLeftJoint>
+                <driveRightJoint>${drive_joint_right}</driveRightJoint>
+                <!-- Wheelbase: distance between the front steering wheel and the rear drive wheels -->
+                <wheelBase>${wheelbase}</wheelBase>
+                <!-- Wheel radius: radius of the rear drive wheels -->
+                <wheelRadius>${wheel_radius}</wheelRadius>
+                <!-- Maximum steering angle, in radians -->
+                <steeringLimit>${steering_limit}</steeringLimit>
+                <!-- Command topic to receive velocity commands -->
+                <commandTopic>${cmdtopic}</commandTopic>
+                <!-- Topic to publish odometry messages -->
+                <odometryTopic>${odomtopic}</odometryTopic>
+                <!-- The base frame of the robot (usually the chassis) -->
+                <robotBaseFrame>${chassis}</robotBaseFrame>
+                <!-- Update rate in Hz -->
+                <updateRate>${update_rate}</updateRate>
+                <!-- Odometry calculation mode: 0 for ENCODER, 1 for WORLD -->
+                <odometrySource>world</odometrySource>
+                <!-- Set to true to publish transforms for the wheel links, defaults to false -->
+                <publishWheelTF>true</publishWheelTF>
+                <!-- Set to true to publish transforms for the odometry, defaults to true -->
+                <publishOdomTF>true</publishOdomTF>
+                <!-- Set to true to swap right and left wheels, defaults to false -->
+                <legacyMode>false</legacyMode>
+            </plugin>
+        </gazebo>
+    </xacro:macro>
     <!-- Macro Template -->
     <!-- <xacro:macro name="robot_link" params="name:=MyRobot m:=1 w:=1 l:=1 h:=1 *first *second **vis **col **ine">

Commit message: feat: ackermann drive plugin xacro

File: urdf/snippets.urdf.xacro (robot description, xacro)
@@ -568,4 +568,35 @@
         </gazebo>
     </xacro:macro>
+    <!-- Ackermann Drive (Ackermann Steering):
+    Ackermann drive system, which is commonly used for car-like
+    steering robots. Ackermann steering model, allows for more
+    realistic simulation of car-like steering where the front
+    wheels pivot while the rear wheels propel the vehicle.
+    https://docs.ros.org/en/rolling/p/gazebo_plugins/generated/classgazebo__plugins_1_1GazeboRosAckermannDrive.html
+    -->
+    <xacro:macro name="robot_drive_ackermann" params="chassis:=base_link front_steer:=joint_chassis_front_steering rear_left:=joint_chassis_rear_left_wheel rear_right:=joint_chassis_rear_right_wheel wheelbase:=1.0 track:=0.5 wheel_radius:=0.15 cmdtopic:=/cmd_vel odomtopic:=/odom max_steering_angle:=0.5 max_speed:=2.0">
+        <gazebo>
+            <plugin name="ackermann_drive_controller" filename="libgazebo_ros_ackermann_drive.so">
+                <!-- Robot links and geometry -->
+                <robotBaseFrame>${chassis}</robotBaseFrame>
+                <steeringJoint>${front_steer}</steeringJoint>
+                <leftRearWheelJoint>${rear_left}</leftRearWheelJoint>
+                <rightRearWheelJoint>${rear_right}</rightRearWheelJoint>
+                <wheelBase>${wheelbase}</wheelBase>
+                <trackWidth>${track}</trackWidth>
+                <wheelRadius>${wheel_radius}</wheelRadius>
+                <!-- Control Topics -->
+                <commandTopic>${cmdtopic}</commandTopic>
+                <odometryTopic>${odomtopic}</odometryTopic>
+                <!-- Limits and Control -->
+                <maxSteeringAngle>${max_steering_angle}</maxSteeringAngle> <!-- Maximum steering angle in radians -->
+                <maxSpeed>${max_speed}</maxSpeed>                         <!-- Maximum linear speed in meters per second -->
+                <updateRate>50</updateRate>                               <!-- Control update rate in Hz -->
+                <!-- Additional configurations -->
+                <publishOdometry>true</publishOdometry>                   <!-- Whether to publish odometry data -->
+                <publishWheelTF>false</publishWheelTF>                    <!-- Whether to publish wheel transforms -->
+            </plugin>
+        </gazebo>
+    </xacro:macro>
     <!-- Macro Template -->
     <!-- <xacro:macro name="robot_link" params="name:=MyRobot m:=1 w:=1 l:=1 h:=1 *first *second **vis **col **ine">
